File: src/eletrica/placa_alimentação_v1.0.1/placa_alimentacao.kicad_sch (KiCad schematic)
At the start: 26 parts, among them J1 XT60-M, J10 22-03-5035, J2 XT60-M, J3 22-03-5035, J4 22-03-5035, J5 22-03-5035, J6 22-03-5035, J7 22-03-5035, J8 22-03-5035, J9 22-03-5035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

Commit message: feat: placa 1.1
Connections:
- net GND: now also J1.N (NEG); no longer J1.P (POS)
- net Vin: now also J1.P (POS); no longer J1.N (NEG)
Other:
- moved on the sheet: J1
Changed lines of the file:
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@@
     (pin "3")
   )
-  (symbol (lib_id "XT-60:XT60-M") (at 25.4 76.2 180) (unit 1)
+  (symbol (lib_id "XT-60:XT60-M") (at 25.4 78.74 0) (mirror y) (unit 1)
     (in_bom yes) (on_board yes) (fields_autoplaced)
     (property "Reference" "J1" (id 0) (at 21.59 68.58 0))
     (property "Value" "XT60-M" (id 1) (at 21.59 71.12 0))
-    (property "Footprint" "AMASS_XT60-M" (id 2) (at 25.4 76.2 0)
+    (property "Footprint" "AMASS_XT60-M" (id 2) (at 25.4 78.74 0)
       (effects (font (size 1.27 1.27)) (justify bottom) hide)
     )
-    (property "Datasheet" "" (id 3) (at 25.4 76.2 0)
+    (property "Datasheet" "" (id 3) (at 25.4 78.74 0)
       (effects (font (size 1.27 1.27)) hide)
     )
-    (property "PARTREV" "V1.2" (id 4) (at 25.4 76.2 0)
+    (property "PARTREV" "V1.2" (id 4) (at 25.4 78.74 0)
       (effects (font (size 1.27 1.27)) (justify bottom) hide)
     )
-    (property "MAXIMUM_PACKAGE_HEIGHT" "16.00 mm" (id 5) (at 25.4 76.2 0)
+    (property "MAXIMUM_PACKAGE_HEIGHT" "16.00 mm" (id 5) (at 25.4 78.74 0)
       (effects (font (size 1.27 1.27)) (justify bottom) hide)
     )
-    (property "STANDARD" "IPC 7351B" (id 6) (at 25.4 76.2 0)
+    (property "STANDARD" "IPC 7351B" (id 6) (at 25.4 78.74 0)
       (effects (font (size 1.27 1.27)) (justify bottom) hide)
     )
-    (property "MANUFACTURER" "AMASS" (id 7) (at 25.4 76.2 0)
+    (property "MANUFACTURER" "AMASS" (id 7) (at 25.4 78.74 0)
       (effects (font (size 1.27 1.27)) (justify bottom) hide)
     )

Commit message: feat: gerber files
Parts:
- J1, J2: footprint AMASS_XT60-M -> XT-60:AMASS_XT60-M
Changed lines of the file:
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@@
     (pin "3")
+  )
+  (symbol (lib_id "EDROM:LOGO") (at 166.37 132.08 0) (unit 1)
+    (in_bom yes) (on_board yes)
+    (property "Reference" "#G1" (id 0) (at 166.37 127.7171 0)
+      (effects (font (size 1.27 1.27)) hide)
+    )
+    (property "Value" "LOGO" (id 1) (at 166.37 136.4429 0)
+      (effects (font (size 1.27 1.27)) hide)
+    )
+    (property "Footprint" "EDROM:LOGO" (id 2) (at 166.37 132.08 0)
+      (effects (font (size 1.27 1.27)) hide)
+    )
+    (property "Datasheet" "" (id 3) (at 166.37 132.08 0)
+      (effects (font (size 1.27 1.27)) hide)
+    )
   )
   (symbol (lib_id "Device:LED") (at 50.8 91.44 90) (unit 1)
@@
     (property "Reference" "J1" (id 0) (at 21.59 68.58 0))
     (property "Value" "XT60-M" (id 1) (at 21.59 71.12 0))
-    (property "Footprint" "AMASS_XT60-M" (id 2) (at 25.4 78.74 0)
+    (property "Footprint" "XT-60:AMASS_XT60-M" (id 2) (at 25.4 78.74 0)
       (effects (font (size 1.27 1.27)) (justify bottom) hide)
     )
@@
       (effects (font (size 1.27 1.27)) (justify bottom) hide)
     )
+    (property "Field8" "" (id 8) (at 25.4 78.74 0))
     (pin "N")
     (pin "P")
@@
     (pin "2")
   )
-  (symbol (lib_id "XT-60:XT60-M") (at 223.52 67.31 0) (unit 1)
+  (symbol (lib_name "XT60-M_1") (lib_id "XT-60:XT60-M") (at 223.52 67.31 0) (unit 1)
     (in_bom yes) (on_board yes) (fields_autoplaced)
     (property "Reference" "J2" (id 0) (at 232.41 64.7699 0)
@@
       (effects (font (size 1.27 1.27)) (justify left))
     )
-    (property "Footprint" "AMASS_XT60-M" (id 2) (at 223.52 67.31 0)
+    (property "Footprint" "XT-60:AMASS_XT60-M" (id 2) (at 223.52 67.31 0)
       (effects (font (size 1.27 1.27)) (justify bottom) hide)
     )
@@
       (effects (font (size 1.27 1.27)) (justify bottom) hide)
     )
+    (property "Field8" "" (id 8) (at 223.52 67.31 0))
     (pin "N")
     (pin "P")
@@
   )
   (symbol_instances
+    (path "/3c20a6f1-3eb7-4c4c-9457-99e57d50b942"
+      (reference "#G1") (unit 1) (value "LOGO") (footprint "EDROM:LOGO")
+    )
     (path "/d00ff660-7bec-49ff-9630-fec487e92632"
       (reference "C1") (unit 1) (value "4700uF") (footprint "Capacitor_THT:CP_Radial_D6.3mm_P2.50mm")
@@
     )
     (path "/c64a0660-3bb4-4b8e-b270-bd72051e9faf"
-      (reference "J1") (unit 1) (value "XT60-M") (footprint "AMASS_XT60-M")
+      (reference "J1") (unit 1) (value "XT60-M") (footprint "XT-60:AMASS_XT60-M")
     )
     (path "/f66ee366-8ba7-428e-8ff7-3797c6acfc22"
-      (reference "J2") (unit 1) (value "XT60-M") (footprint "AMASS_XT60-M")
+      (reference "J2") (unit 1) (value "XT60-M") (footprint "XT-60:AMASS_XT60-M")
     )
     (path "/c3e8912f-0491-4f67-b4ba-2e52728b7346"
