Commit message: Atualização do modelo da robô nova e de seu urdf.

File: src/movement_bioloid/humanoid_visualization/urdf/nova.urdf (robot description, URDF)
Before this commit: robot nova, 19 links, 18 joints
Links:
- link LFOOT: geometry visual box size=0.13 0.08 0.002
- link RFOOT: geometry visual box size=0.13 0.08 0.002
Joints:
- joint LANKLE_UX_joint: origin xyz=-0.073 0 0 rpy=0 0 0 -> xyz=0 0 0 rpy=0 0 0
- joint LANKLE_UY_joint: origin xyz=0 0 -0.083 rpy=0 0 0 -> xyz=0.0083 0 -0.08 rpy=0 0 0
- joint LFOOT_joint: origin xyz=0.05 0 -0.028 rpy=0 0 0 -> xyz=-0.021 0 -0.029 rpy=0 0 0
- joint LHIP_UX_joint: origin xyz=-0.051 0 -0.034 rpy=0 0 0 -> xyz=0.021 0 -0.02882 rpy=0 0 0
- joint LHIP_UY_joint: origin xyz=0.073 0 0 rpy=0 0 0 -> xyz=0 0 0 rpy=0 0 0
- joint LHIP_UZ_joint: origin xyz=0.002 0.042 -0.045 rpy=0 0 0 -> xyz=0.0025 0.0425 -0.0468 rpy=0 0 0
- joint LKNEE_joint: origin xyz=0 0 -0.11 rpy=0 0 0 -> xyz=0 0 -0.1111 rpy=0 0 0
- joint RANKLE_UX_joint: origin xyz=-0.073 0 0 rpy=0 0 0 -> xyz=0 0 0 rpy=0 0 0
- joint RANKLE_UY_joint: origin xyz=0 0 -0.083 rpy=0 0 0 -> xyz=0.0083 0 -0.08 rpy=0 0 0
- joint RFOOT_joint: origin xyz=0.05 0 -0.028 rpy=0 0 0 -> xyz=-0.021 0 -0.029 rpy=0 0 0
- joint RHIP_UX_joint: origin xyz=-0.051 0 -0.034 rpy=0 0 0 -> xyz=0.021 0 -0.02882 rpy=0 0 0
- joint RHIP_UY_joint: origin xyz=0.073 0 0 rpy=0 0 0 -> xyz=0 0 0 rpy=0 0 0
- joint RHIP_UZ_joint: origin xyz=0.002 -0.042 -0.045 rpy=0 0 0 -> xyz=0.0025 -0.0425 -0.0468 rpy=0 0 0
- joint RKNEE_joint: origin xyz=0 0 -0.11 rpy=0 0 0 -> xyz=0 0 -0.1111 rpy=0 0 0
- joint base_to_COM: origin xyz=0 0 0.295 -> xyz=0 0 0.29846
