Commit message: Revisão da caminhada - tunagem de parametros

File: src/movement/humanoid_visualization/urdf/aurea.urdf (robot description, URDF)
Before this commit: robot aurea, 19 links, 18 joints
Joints:
- joint LANKLE_UX_joint: axis 1 0 0 -> -1 0 0
- joint LHIP_UZ_joint: axis 0 0 1 -> 0 0 -1
- joint LKNEE_joint: axis 0 1 0 -> 0 -1 0
- joint RANKLE_UX_joint: axis 1 0 0 -> -1 0 0
- joint RHIP_UY_joint: axis 0 1 0 -> 0 -1 0
- joint RHIP_UZ_joint: axis 0 0 1 -> 0 0 -1
- joint RKNEE_joint: axis 0 1 0 -> 0 -1 0

Commit message: Criação de código falso da u2d2 para eliminar necessidade de plugar a robô em testes básicos e/ou de visualização, implementação das correções aplicadas no COM do modelo (.json) da robô na visualização, alteração do esquema de funcionamento para atualização do modelo da robô na core (Agora é chamado após qualquer comando na core, utilizando a última posição enviada para os motores como base, antes da publicação para visualização para que esta siga o modelo instantaneamente). Ou seja, foi removida a necessidade de pedir feedback, o que DEVE ser avaliado, talvez parar de pedir o tempo todo e só eventualmente (timer) para acertar o modelo com o real.

File: src/movement/humanoid_visualization/urdf/aurea.urdf (robot description, URDF)
Before this commit: robot aurea, 19 links, 18 joints
Links:
- added link COM_height
- added link COM_pitch
Joints:
- added joint COM_height_slider: type prismatic, parent base_link, child COM_height, origin xyz=0 0 0.29846, axis 0 0 1, limit lower=-1 upper=1 effort=1000.0 velocity=10
- added joint COM_pitch_joint: type revolute, parent COM_height, child COM_pitch, origin xyz=0 0 0, axis 0 1 0, limit lower=-3.14 upper=3.14 effort=1000.0 velocity=10
- joint base_to_COM: origin xyz=0 0 0.29846 -> xyz=0 0 0; parent base_link -> COM_pitch
