Commit message: update sim

File: src/movement/Ros2_change/src/urdf_robox/urdf/urdf_robox.urdf (robot description, URDF)
Before this commit: robot urdf_robox, 31 links, 30 joints
Links:
- added link world
Joints:
- added joint base_joint: type fixed, parent world, child Link_0, origin xyz=0 0 0.40
- joint LANKLE_UY2: mimic (none) -> joint=LANKLE_UY1 multiplier=1 offset=0
- joint LANKLE_UY3: mimic (none) -> joint=LANKLE_UY1 multiplier=1 offset=0
- joint LHIP_UY2: axis 0 -1 0 -> 0 1 0; mimic (none) -> joint=LHIP_UY1 multiplier=1 offset=0
- joint LHIP_UY3: mimic (none) -> joint=LHIP_UY1 multiplier=1 offset=0
- joint LLKNEE_2: mimic (none) -> joint=LLKNEE_1 multiplier=1 offset=0
- joint LLKNEE_3: mimic (none) -> joint=LLKNEE_1 multiplier=1 offset=0
- joint LUKNEE_2: mimic (none) -> joint=LUKNEE_1 multiplier=1 offset=0
- joint LUKNEE_3: mimic (none) -> joint=LUKNEE_1 multiplier=1 offset=0
- joint RANKLE_UY2: mimic (none) -> joint=RANKLE_UY1 multiplier=1 offset=0
- joint RANKLE_UY3: mimic (none) -> joint=RANKLE_UY1 multiplier=1 offset=0
- joint RHIP_UY2: axis 0 -1 0 -> 0 1 0; mimic (none) -> joint=RHIP_UY1 multiplier=1 offset=0
- joint RHIP_UY3: mimic (none) -> joint=RHIP_UY1 multiplier=1 offset=0
- joint RLKNEE_2: mimic (none) -> joint=RLKNEE_1 multiplier=1 offset=0
- joint RLKNEE_3: mimic (none) -> joint=RLKNEE_1 multiplier=1 offset=0
- joint RUKNEE_2: mimic (none) -> joint=RUKNEE_1 multiplier=1 offset=0
- joint RUKNEE_3: mimic (none) -> joint=RUKNEE_1 multiplier=1 offset=0
